Commit message: Mid test

File: urdf/boat.urdf (robot description, URDF)
Before this commit: robot csi_cam_0, 2 links, 1 joints
Links:
- removed link optical_frame
- added link cg_ned
- added link csi_cam_0_link
Joints:
- added joint pixhawk_transform: type fixed, parent base_link, child cg_ned, origin xyz=0.15 0 0 rpy=3.14159 0 -1.57079
- joint optical_frame_to_base: child optical_frame -> csi_cam_0_link; origin (none) -> xyz=0 0 0 rpy=0 1.57079 0

Commit message: Working RC override.
Need to add rosservice calls to set SERVOX_FUNCTION parameter.

File: urdf/boat.urdf (robot description, URDF)
Before this commit: robot boat, 3 links, 2 joints
Joints:
- joint optical_frame_to_base: origin xyz=0 0 0 rpy=0 1.57079 0 -> xyz=0 0 -0.08 rpy=0 1.5708 0; parent base_link -> cg_ned
- joint pixhawk_transform: origin xyz=0.15 0 0 rpy=3.14159 0 -1.57079 -> xyz=-0.15 0 0 rpy=3.14159 0 0

Commit message: Dock trasform working. Position hold based on cg_ned frame

File: urdf/boat.urdf (robot description, URDF)
Before this commit: robot boat, 3 links, 2 joints
Links:
- link cg_ned: geometry visual mesh filename=file:///home/alec/PycharmProjects/boat_ws/src/docking_contr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 scale=0.001 0.001 0.001
Joints:
- joint optical_frame_to_base: origin xyz=0 0 -0.08 rpy=0 1.5708 0 -> xyz=-0.03 0 -0.09 rpy=1.5708 0 1.5708

Commit message: Updated AR tags work in pool

File: urdf/boat.urdf (robot description, URDF)
Before this commit: robot boat, 3 links, 2 joints
Links:
- added link imu
Joints:
- added joint imu_to_base: type fixed, parent cg_ned, child imu, origin xyz=0 0 0 rpy=0 0 0

Commit message: Added derivative tracking for angular velocity. This worked much better for following paths

File: urdf/boat.urdf (robot description, URDF)
Before this commit: robot boat, 4 links, 3 joints
Joints:
- joint imu_to_base: origin xyz=0 0 0 rpy=0 0 0 -> xyz=0 0 0 rpy=0 3.14159 0
